File: rotary-breakout/rotary-breakout.kicad_pcb (KiCad board)
At the start: 2 copper layers, 28.4 x 24.4 mm, 9 parts, among them J1 CONN_01X05

Commit message: Combine libraries
Parts:
- ROT1: footprint lci-relays:Alps-Rotary-Encoder -> lci-kicad:Alps-Rotary-Encoder
Changed lines of the file:
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@@
-(kicad_pcb (version 4) (host pcbnew 4.0.7)
+(kicad_pcb (version 20171130) (host pcbnew "(5.0.0-rc2-dev-310-g1cd6477)")
   (general
-    (links 11)
-    (no_connects 0)
-    (area 131.7399 70.214166 173.888001 97.463)
     (thickness 1.6)
     (drawings 12)
@@
       (layerselection 0x00030_80000001)
       (usegerberextensions false)
+      (usegerberattributes false)
+      (usegerberadvancedattributes false)
+      (creategerberjobfile false)
       (excludeedgelayer true)
       (linewidth 0.100000)
@@
       (hpglpenspeed 20)
       (hpglpendiameter 15)
-      (hpglpenoverlay 2)
       (psnegative false)
       (psa4output false)
@@
     (add_net VCC)
   )
+  (module lci-kicad:Alps-Rotary-Encoder (layer F.Cu)
+    (at 142.24 84.328 270)
+    (fp_text reference ROT1 (at 0 9.5 270) (layer F.SilkS)
+      (effects (font (size 0.762 0.762) (thickness 0.1524)))
+    )
+    (fp_text value Alps-Rotary-Encoder (at 0 0 270) (layer F.SilkS) hide
+      (effects (font (size 0.762 0.762) (thickness 0.1524)))
+    )
+    (fp_line (start 6 -6.5) (end 6 6.5) (layer F.SilkS) (width 0.2032))
+    (fp_line (start -6 -6.5) (end 6 -6.5) (layer F.SilkS) (width 0.2032))
+    (fp_line (start -6 6.5) (end -6 -6.5) (layer F.SilkS) (width 0.2032))
+    (fp_line (start 6 6.5) (end -6 6.5) (layer F.SilkS) (width 0.2032))
+    (fp_circle (center 0 0) (end 3.5 0) (layer F.SilkS) (width 0.2032))
+    (fp_line (start 3 -1.5) (end -3 -1.5) (layer F.SilkS) (width 0.2032))
+    (pad "" thru_hole circle (at -5.6 0 270) (size 3 3) (drill 2.2) (layers *.Cu *.Mask F.SilkS))
+    (pad "" thru_hole circle (at 5.6 0 270) (size 3 3) (drill 2.2) (layers *.Cu *.Mask F.SilkS))
+    (pad 5 thru_hole circle (at 2.5 -7 270) (size 1.8 1.8) (drill 1) (layers *.Cu *.Mask F.SilkS)
+      (net 3 "Net-(J1-Pad3)"))
+    (pad 4 thru_hole circle (at 2.5 7.5 270) (size 1.8 1.8) (drill 1) (layers *.Cu *.Mask F.SilkS)
+      (net 2 "Net-(J1-Pad2)"))
+    (pad 3 thru_hole circle (at 0 7.5 270) (size 1.8 1.8) (drill 1) (layers *.Cu *.Mask F.SilkS)
+      (net 4 GND))
+    (pad 2 thru_hole circle (at -2.5 7.5 270) (size 1.8 1.8) (drill 1) (layers *.Cu *.Mask F.SilkS)
+      (net 1 "Net-(J1-Pad1)"))
+    (pad 1 thru_hole circle (at -2.5 -7 270) (size 1.8 1.8) (drill 1) (layers *.Cu *.Mask F.SilkS)
+      (net 4 GND))
+  )
   (module Resistors_SMD:R_0603_HandSoldering (layer B.Cu)
     (at 137.668 83.312 90)
@@
       (rotate (xyz 0 0 0))
     )
-  )
-  (module lci-relays:Alps-Rotary-Encoder (layer F.Cu)
-    (at 142.24 84.328 270)
-    (fp_text reference ROT1 (at 0 9.5 270) (layer F.SilkS)
-      (effects (font (size 0.762 0.762) (thickness 0.1524)))
-    )
-    (fp_text value Alps-Rotary-Encoder (at 0 0 270) (layer F.SilkS) hide
-      (effects (font (size 0.762 0.762) (thickness 0.1524)))
-    )
-    (fp_line (start 3 -1.5) (end -3 -1.5) (layer F.SilkS) (width 0.2032))
-    (fp_circle (center 0 0) (end 3.5 0) (layer F.SilkS) (width 0.2032))
-    (fp_line (start 6 6.5) (end -6 6.5) (layer F.SilkS) (width 0.2032))
-    (fp_line (start -6 6.5) (end -6 -6.5) (layer F.SilkS) (width 0.2032))
-    (fp_line (start -6 -6.5) (end 6 -6.5) (layer F.SilkS) (width 0.2032))
-    (fp_line (start 6 -6.5) (end 6 6.5) (layer F.SilkS) (width 0.2032))
-    (pad 1 thru_hole circle (at -2.5 -7 270) (size 1.8 1.8) (drill 1) (layers *.Cu *.Mask F.SilkS)
-      (net 4 GND))
-    (pad 2 thru_hole circle (at -2.5 7.5 270) (size 1.8 1.8) (drill 1) (layers *.Cu *.Mask F.SilkS)
-      (net 1 "Net-(J1-Pad1)"))
-    (pad 3 thru_hole circle (at 0 7.5 270) (size 1.8 1.8) (drill 1) (layers *.Cu *.Mask F.SilkS)
-      (net 4 GND))
-    (pad 4 thru_hole circle (at 2.5 7.5 270) (size 1.8 1.8) (drill 1) (layers *.Cu *.Mask F.SilkS)
-      (net 2 "Net-(J1-Pad2)"))
-    (pad 5 thru_hole circle (at 2.5 -7 270) (size 1.8 1.8) (drill 1) (layers *.Cu *.Mask F.SilkS)
-      (net 3 "Net-(J1-Pad3)"))
-    (pad "" thru_hole circle (at 5.6 0 270) (size 3 3) (drill 2.2) (layers *.Cu *.Mask F.SilkS))
-    (pad "" thru_hole circle (at -5.6 0 270) (size 3 3) (drill 2.2) (layers *.Cu *.Mask F.SilkS))
   )
   (module Pin_Headers:Pin_Header_Straight_1x05_Pitch2.54mm (layer F.Cu)
@@
       (net 5 VCC))
     (model Pin_Headers.3dshapes/Pin_Header_Straight_1x05_Pitch2.54mm.wrl
-      (at (xyz 0 -0.2 0))
+      (offset (xyz 0 -5.079999923706055 0))
       (scale (xyz 1 1 1))
       (rotate (xyz 0 0 90))
