File: 3-way-class-d/3-way-class-d.sch (KiCad schematic (older format))
At the start: 0 parts

Commit message: More input
Changed lines of the file:
@@
 S 2550 3100 1550 1200
 U 57A9B7AF
-F0 "Input" 60
-F1 "Input.sch" 60
+F0 "input" 60
+F1 "input.sch" 60
 $EndSheet
 $EndSCHEMATC

Commit message: ADC
Changed lines of the file:
@@
 LIBS:conn
 LIBS:transistors
-LIBS:texas
 LIBS:digital-audio
 LIBS:analog_switches
 LIBS:device
 LIBS:lci-kicad
+LIBS:linear
 LIBS:3-way-class-d-cache
 EELAYER 25 0
@@
 $Descr A4 11693 8268
 encoding utf-8
-Sheet 1 3
+Sheet 1 4
 Title ""
 Date ""
@@
 $EndSheet
 $Sheet
-S 2550 3100 1550 1200
+S 2600 4950 1550 1200
 U 57A9B7AF
 F0 "input" 60
 F1 "input.sch" 60
 $EndSheet
+$Sheet
+S 2550 1250 1500 1200
+U 58C18DAC
+F0 "analog input" 60
+F1 "analog.sch" 60
+$EndSheet
 $EndSCHEMATC
