File: 3-way-class-d/analog.sch (KiCad schematic (older format))
At the start: 23 parts, among them U4 CS5361

Commit message: Add peak_detect
Parts:
- added D?: LED, symbol Led_Small
- added R?: 470, symbol R_Small
Connections:
- net +3V3: now also R?.1
- net at U4.15 (~OVFL): now also D?.1 (K)
- new net: D?.2 (A), R?.2
Other:
- note added: "overflow"
Changed lines of the file:
@@
 	1    0    0    -1
 $EndComp
-Text GLabel 9300 4050 2    60   Input ~ 12
+Text GLabel 9300 4050 2    60   Output ~ 12
 LRCLK
-Text GLabel 9700 4150 2    60   Input ~ 12
+Text GLabel 9700 4150 2    60   Output ~ 12
 SCLK
-Text GLabel 10050 4250 2    60   Input ~ 12
+Text GLabel 10050 4250 2    60   Output ~ 12
 MCLK
 $Comp
@@
 	1    0    0    -1
 $EndComp
+$Comp
+L Led_Small D?
+U 1 1 58C2FA90
+P 9900 3250
+F 0 "D?" H 9850 3375 50  0000 L CNN
+F 1 "LED" H 9850 3150 50  0000 L CNN
+F 2 "" V 9900 3250 60  0000 C CNN
+F 3 "" V 9900 3250 60  0000 C CNN
+	1    9900 3250
+	1    0    0    -1
+$EndComp
+$Comp
+L R_Small R?
+U 1 1 58C2FB7F
+P 10100 3250
+F 0 "R?" H 10130 3270 50  0000 L CNN
+F 1 "470" H 10130 3210 50  0000 L CNN
+F 2 "" H 10100 3250 60  0000 C CNN
+F 3 "" H 10100 3250 60  0000 C CNN
+	1    10100 3250
+	0    1    1    0
+$EndComp
+Wire Wire Line
+	9150 3250 9800 3250
+$Comp
+L +3.3V #PWR?
+U 1 1 58C30782
+P 10200 3250
+F 0 "#PWR?" H 10200 3100 50  0001 C CNN
+F 1 "+3.3V" H 10200 3390 50  0000 C CNN
+F 2 "" H 10200 3250 60  0000 C CNN
+F 3 "" H 10200 3250 60  0000 C CNN
+	1    10200 3250
+	0    1    1    0
+$EndComp
+Text Notes 9850 3550 0    60   ~ 0
+overflow
+Wire Notes Line
+	9800 3000 10450 3000
+Wire Notes Line
+	10450 3000 10450 3600
+Wire Notes Line
+	10450 3600 9800 3600
+Wire Notes Line
+	9800 3600 9800 3000
 $EndSCHEMATC

Commit message: Update remaining projects to KiCad 5
Parts:
- C? (x2): symbol RCA -> lci-kicad:RCA
- C? (x13): symbol C_Small -> device:C_Small
- D?: symbol Led_Small -> device:LED_Small
- R? (x5): symbol R_Small -> device:R_Small
- U4: symbol CS5361 -> digital-audio:CS5361
- U? (x2): symbol OPA2340 -> linear:OPA2340
- U?: symbol TLE2426 -> lci-kicad:TLE2426
Connections:
- wire segments 87 -> 109
