File: 3-way-class-d/class-d.sch (KiCad schematic (older format))
At the start: 88 parts, among them P1 CONN_02X02, P2 CONN_02X03, Q1 BC857, Q2 BC857, Q3 BC857, U1 TAS5701

Commit message: Update remaining projects to KiCad 5
Parts:
- C1, C10, C11, C12, C13, C14, C15, C16, C17, C18, C19, C2, C20, C21, C22, C23, C24, C25, C26, C27, C28, C29, C3, C30, C31, C32, C33, C34, C35, C36, C37, C38, C39, C4, C40, C41, C42, C43, C44, C45, C46, C47, C48, C5, C6, C7, C8, C9: symbol C -> device:C
- D1: symbol LED -> device:LED
- D2, D3: symbol LED -> device:LED_Small
- L1, L2, L3, L4: symbol INDUCTOR -> device:L
- P1: symbol CONN_02X02 -> Connector:Conn_02x02_Odd_Even
- P2: symbol CONN_02X03 -> Connector:Conn_02x03_Odd_Even
- Q1, Q2, Q3: symbol BC857 -> Transistor:BC857
- R1, R10, R11, R12, R13, R14, R15, R16, R17, R18, R19, R2, R20, R21, R22, R23, R24, R25, R26, R27, R3, R4, R5, R6, R7, R8, R9: symbol R -> device:R
- U1: symbol TAS5701 -> lci-kicad:TAS5701
