File: usb-switch/usb-switch.kicad_pcb (KiCad board)
At the start: 2 copper layers, 38.1 x 17.8 mm, 11 parts, among them IC1 4N25, P1 input, P2 power, P3 output, Q1 BC307

Commit message: Update remaining projects to KiCad 5
Parts:
- removed REF** (x2): 1pin, Connect:1pin
Connections:
- IC1 pad 3: (no net) -> Net-(IC1-Pad3)
- IC1 pad 6: (no net) -> Net-(IC1-Pad6)
- RL1 pad 5: (no net) -> Net-(RL1-Pad5)
- RL1 pad 6: (no net) -> Net-(RL1-Pad6)
- RL1 pad 7: (no net) -> Net-(RL1-Pad7)
Changed lines of the file:
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@@
-(kicad_pcb (version 4) (host pcbnew "(2015-01-07 BZR 5357)-product")
+(kicad_pcb (version 20171130) (host pcbnew "(5.0.0-rc2-dev-310-g1cd6477)")
   (general
-    (links 15)
-    (no_connects 0)
-    (area 21.514999 17.363 59.765001 40.419)
     (thickness 1.6)
     (drawings 4)
     (tracks 50)
     (zones 0)
-    (modules 11)
-    (nets 12)
+    (modules 9)
+    (nets 17)
   )
   (page A4 portrait)
@@
       (usegerberextensions true)
       (usegerberattributes true)
+      (usegerberadvancedattributes false)
+      (creategerberjobfile false)
       (excludeedgelayer true)
       (linewidth 0.100000)
@@
       (hpglpenspeed 20)
       (hpglpendiameter 15)
-      (hpglpenoverlay 2)
       (psnegative false)
       (psa4output false)
@@
   (net 10 "Net-(FB1-Pad3)")
   (net 11 "Net-(FB1-Pad4)")
+  (net 12 "Net-(RL1-Pad7)")
+  (net 13 "Net-(RL1-Pad6)")
+  (net 14 "Net-(RL1-Pad5)")
+  (net 15 "Net-(IC1-Pad3)")
+  (net 16 "Net-(IC1-Pad6)")
   (net_class Default "This is the default net class."
     (clearance 0.254)
@@
     (add_net "Net-(IC1-Pad1)")
     (add_net "Net-(IC1-Pad2)")
+    (add_net "Net-(IC1-Pad3)")
     (add_net "Net-(IC1-Pad5)")
+    (add_net "Net-(IC1-Pad6)")
     (add_net "Net-(P1-Pad1)")
     (add_net "Net-(Q1-Pad1)")
     (add_net "Net-(Q1-Pad2)")
+    (add_net "Net-(RL1-Pad5)")
+    (add_net "Net-(RL1-Pad6)")
+    (add_net "Net-(RL1-Pad7)")
   )
   (net_class Wide ""
@@
       (net 2 "Net-(IC1-Pad2)"))
     (model Pin_Headers.3dshapes/Pin_Header_Straight_1x02.wrl
-      (at (xyz 0 -0.05 0))
+      (offset (xyz 0 -1.269999980926514 0))
       (scale (xyz 1 1 1))
       (rotate (xyz 0 0 90))
@@
       (net 11 "Net-(FB1-Pad4)"))
     (model Pin_Headers.3dshapes/Pin_Header_Straight_1x02.wrl
-      (at (xyz 0 -0.05 0))
+      (offset (xyz 0 -1.269999980926514 0))
       (scale (xyz 1 1 1))
       (rotate (xyz 0 0 90))
@@
       (net 3 GND))
     (model Pin_Headers.3dshapes/Pin_Header_Straight_1x02.wrl
-      (at (xyz 0 -0.05 0))
+      (offset (xyz 0 -1.269999980926514 0))
       (scale (xyz 1 1 1))
       (rotate (xyz 0 0 90))
@@
       (net 9 "Net-(Q1-Pad1)"))
     (model Housings_TO-92.3dshapes/TO-92_Inline_Narrow_Oval.wrl
-      (at (xyz 0.05 0 0))
+      (offset (xyz 1.269999980926514 0 0))
       (scale (xyz 1 1 1))
       (rotate (xyz 0 0 -90))
@@
     (pad 2 thru_hole circle (at 0 3.81 90) (size 1.397 1.397) (drill 0.8128) (layers *.Cu *.Mask F.SilkS)
       (net 2 "Net-(IC1-Pad2)"))
-    (pad 3 thru_hole circle (at 2.54 3.81 90) (size 1.397 1.397) (drill 0.8128) (layers *.Cu *.Mask F.SilkS))
+    (pad 3 thru_hole circle (at 2.54 3.81 90) (size 1.397 1.397) (drill 0.8128) (layers *.Cu *.Mask F.SilkS)
+      (net 15 "Net-(IC1-Pad3)"))
     (pad 4 thru_hole circle (at 2.54 -3.81 90) (size 1.397 1.397) (drill 0.8128) (layers *.Cu *.Mask F.SilkS)
       (net 3 GND))
     (pad 5 thru_hole circle (at 0 -3.81 90) (size 1.397 1.397) (drill 0.8128) (layers *.Cu *.Mask F.SilkS)
       (net 4 "Net-(IC1-Pad5)"))
-    (pad 6 thru_hole circle (at -2.54 -3.81 90) (size 1.397 1.397) (drill 0.8128) (layers *.Cu *.Mask F.SilkS))
+    (pad 6 thru_hole circle (at -2.54 -3.81 90) (size 1.397 1.397) (drill 0.8128) (layers *.Cu *.Mask F.SilkS)
+      (net 16 "Net-(IC1-Pad6)"))
     (model Sockets_DIP.3dshapes/DIP-6__300.wrl
       (at (xyz 0 0 0))
@@
       (rotate (xyz 0 0 0))
     )
-  )
-  (module Connect:1pin (layer F.Cu)
-    (at 24.13 21.59)
-    (descr "module 1 pin (ou trou mecanique de percage)")
-    (tags DEV)
-    (fp_text reference REF** (at 0 -3.048) (layer F.SilkS) hide
-      (effects (font (size 1 1) (thickness 0.15)))
-    )
-    (fp_text value 1pin (at 0 2.794) (layer F.Fab) hide
-      (effects (font (size 1 1) (thickness 0.15)))
-    )
-    (fp_circle (center 0 0) (end 0 -2.286) (layer F.SilkS) (width 0.15))
-    (pad 1 thru_hole circle (at 0 0) (size 4.064 4.064) (drill 3.048) (layers *.Cu *.Mask F.SilkS))
-  )
-  (module Connect:1pin (layer F.Cu)
-    (at 57.15 34.29)
-    (descr "module 1 pin (ou trou mecanique de percage)")
-    (tags DEV)
-    (fp_text reference REF** (at 0 -3.048) (layer F.SilkS) hide
-      (effects (font (size 1 1) (thickness 0.15)))
-    )
-    (fp_text value 1pin (at 0 2.794) (layer F.Fab) hide
-      (effects (font (size 1 1) (thickness 0.15)))
-    )
-    (fp_circle (center 0 0) (end 0 -2.286) (layer F.SilkS) (width 0.15))
-    (pad 1 thru_hole circle (at 0 0) (size 4.064 4.064) (drill 3.048) (layers *.Cu *.Mask F.SilkS))
   )
   (module lci-relays:Omron-G6K (layer F.Cu)
@@
     (pad 8 thru_hole circle (at -3.81 -2.54 180) (size 1.524 1.524) (drill 0.762) (layers *.Cu *.Mask F.SilkS)
       (net 3 GND))
-    (pad 7 thru_hole circle (at -1.27 -2.54 180) (size 1.524 1.524) (drill 0.762) (layers *.Cu *.Mask F.SilkS))
-    (pad 6 thru_hole circle (at 1.27 -2.54 180) (size 1.524 1.524) (drill 0.762) (layers *.Cu *.Mask F.SilkS))
-    (pad 5 thru_hole circle (at 3.81 -2.54 180) (size 1.524 1.524) (drill 0.762) (layers *.Cu *.Mask F.SilkS))
+    (pad 7 thru_hole circle (at -1.27 -2.54 180) (size 1.524 1.524) (drill 0.762) (layers *.Cu *.Mask F.SilkS)
+      (net 12 "Net-(RL1-Pad7)"))
+    (pad 6 thru_hole circle (at 1.27 -2.54 180) (size 1.524 1.524) (drill 0.762) (layers *.Cu *.Mask F.SilkS)
+      (net 13 "Net-(RL1-Pad6)"))
+    (pad 5 thru_hole circle (at 3.81 -2.54 180) (size 1.524 1.524) (drill 0.762) (layers *.Cu *.Mask F.SilkS)
+      (net 14 "Net-(RL1-Pad5)"))
   )
   (module lci-relays:double_choke (layer F.Cu)
