File: P2/P2.kicad_pcb (KiCad board)
At the start: 2 copper layers, 86.4 x 45.7 mm, 32 parts, among them J1 12v, J10 PWR2, J11 r1, J12 r2, J2 Channels, J3 Noritake, J4 POWER, J5 Q, J6 Volume, J7 PGM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

Commit message: Run DRC un P2
Routing:
- net GND: track 75.0 -> 107.0 mm, vias 9 -> 12
- net Net-(U1-Pad3): track 13.5 -> 18.2 mm
- net +5V: track 345.2 -> 346.4 mm
