File: espsense/espsense.kicad_pcb (KiCad board)
At the start: 2 copper layers, 66 x 68.6 mm, 32 parts, among them J1 Conn_01x03_Female, J2 Conn_01x03_Female, J3 Conn_01x02_Female, J4 Conn_01x02_Female, J5 Conn_01x02_Female, J6 Conn_01x06_Male, Q1 Q_NPN_BCE, Q2 Q_NPN_BCE, SW1 SW_SPDT, SW2 SW_SPDT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

Commit message: Fix espsense (phew)
Parts:
- added J7: Conn_01x03_Female, Connector_Wire:SolderWirePad_1x03_P4.445mm_Drill1.5mm, F.Cu at (180.3, 85.3)
- J5: value Conn_01x02_Female -> Conn_01x03_Female; footprint Connector_Wire:SolderWirePad_1x02_P5.08mm_Drill1.5mm -> Connector_Wire:SolderWirePad_1x03_P4.445mm_Drill1.5mm
- moved J3 63.6 mm to (119.4, 104.1), turned to 90 degrees
- moved R6 53.8 mm to (171.7, 117.3), turned to 180 degrees
- moved R3 52.1 mm to (130.1, 117.3)
- moved U2 48.9 mm to (168.1, 113.3)
- moved U1 48.8 mm to (126.5, 114.3)
- moved R5 38.6 mm to (176.3, 107.7), turned to 270 degrees
- moved R2 31.0 mm to (134.6, 108.7), turned to 270 degrees
- moved R4 19.4 mm to (165.6, 108.7), turned to 90 degrees
- moved R1 18.0 mm to (122.4, 114.3)
- moved U4 11.4 mm to (143.3, 124.5), turned to 270 degrees
- moved U3 9.54 mm to (136.1, 126.2)
- moved R7 8.69 mm to (140.2, 112.8), turned to 90 degrees
- moved J1 7.62 mm to (129.0, 75.2), turned to 0 degrees
- moved Q1 6.10 mm to (139.1, 107.2)
- moved SW1 5.24 mm to (131.6, 90.9)
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Connections:
- J1 pad 1: Net-(J1-Pad1) -> Earth_Protective
- J1 pad 2: /SW1 -> GND
- J1 pad 3: Net-(J1-Pad3) -> /SW1
- J2 pad 1: Net-(J2-Pad1) -> Earth_Protective
- J2 pad 2: /SW2 -> GND
- J2 pad 3: Net-(J2-Pad3) -> /SW2
- J5 pad 1: GND -> Earth_Protective
- J5 pad 2: AC -> GND
- J6 pad 3: (no net) -> +3V3
- RL1 pad 3: Net-(J1-Pad3) -> Net-(RL1-Pad3)
- RL1 pad 5: Net-(J1-Pad1) -> Net-(RL1-Pad5)
- RL2 pad 3: Net-(J2-Pad3) -> Net-(RL2-Pad3)
- RL2 pad 5: Net-(J2-Pad1) -> Net-(RL2-Pad5)
- SW1 pad 1: Net-(J1-Pad1) -> Net-(RL1-Pad5)
- SW1 pad 3: Net-(J1-Pad3) -> Net-(RL1-Pad3)
- SW2 pad 1: Net-(J2-Pad1) -> Net-(RL2-Pad5)
- SW2 pad 3: Net-(J2-Pad3) -> Net-(RL2-Pad3)
- U3 pad 2: (no net) -> GNDD
- U3 pad 6: (no net) -> +3V3
Routing:
- net Earth_Protective: track 0.00 -> 76.0 mm
- net Net-(R4-Pad1): track 75.7 -> 5.22 mm, vias 2 -> 0
- net Net-(R1-Pad1): track 71.8 -> 3.03 mm, vias 2 -> 0
- net GND: track 114.0 -> 153.7 mm
- net Net-(J1-Pad3): track 39.1 -> 0.00 mm
- net Net-(J1-Pad1): track 37.7 -> 0.00 mm
- net Net-(J2-Pad1): track 37.5 -> 0.00 mm
- net Net-(J2-Pad3): track 36.8 -> 0.00 mm
- net Net-(R8-Pad2): track 24.9 -> 60.1 mm
- net GNDD: track 70.0 -> 92.4 mm
- net Net-(R6-Pad2): track 24.5 -> 4.06 mm
- net Net-(R3-Pad2): track 20.7 -> 3.05 mm
- net Net-(RL2-Pad3): track 0.00 -> 16.8 mm
- net /SW1: track 34.4 -> 50.1 mm
- net Net-(RL2-Pad5): track 0.00 -> 15.1 mm
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Other:
- board text added: "E"
- board text added: "L"
- board text added: "N"
