File: headphone-power/headphone-power.kicad_pcb (KiCad board)
At the start: 2 copper layers, 57.1 x 34.3 mm, 18 parts, among them J1 Conn_01x02_Female, J2 Conn_01x02_Female, J3 Conn_01x02_Female, U1 LM7815_TO220

Commit message: Fix espsense (phew)
Connections:
- D1 pad 1: Net-(D1-Pad1) -> AC
- D1 pad 2: AC -> Net-(D1-Pad2)
- D2 pad 1: Net-(D1-Pad1) -> AC
- D3 pad 2: AC -> Net-(D1-Pad2)
- J3 pad 2: Net-(D1-Pad1) -> AC
Routing:
- net Net-(D1-Pad1): track 14.4 -> 0.00 mm
- net AC: track 4.06 -> 14.4 mm
- net Net-(D1-Pad2): track 0.00 -> 4.06 mm
Changed lines of the file:
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@@
   )
   (setup
-    (last_trace_width 0.5)
+    (last_trace_width 0.25)
     (user_trace_width 0.5)
     (trace_clearance 0.2)
@@
       (outputformat 1)
       (mirror false)
-      (drillshape 1)
+      (drillshape 0)
       (scaleselection 1)
-      (outputdirectory ""))
+      (outputdirectory "gerber"))
   )
   (net 0 "")
@@
   (net 3 "Net-(C2-Pad2)")
   (net 4 "Net-(C3-Pad2)")
-  (net 5 "Net-(D1-Pad1)")
-  (net 6 AC)
-  (net 7 "Net-(C4-Pad1)")
+  (net 5 AC)
+  (net 6 "Net-(C4-Pad1)")
+  (net 7 "Net-(D1-Pad2)")
   (net_class Default "This is the default net class."
     (clearance 0.2)
@@
     (add_net "Net-(C3-Pad2)")
     (add_net "Net-(C4-Pad1)")
-    (add_net "Net-(D1-Pad1)")
+    (add_net "Net-(D1-Pad2)")
   )
   (module Capacitor_THT:CP_Radial_D10.0mm_P5.00mm_P7.50mm (layer F.Cu)
@@
     )
     (pad 1 thru_hole rect (at 0 0) (size 1.905 2) (drill 1.1) (layers *.Cu *.Mask)
-      (net 7 "Net-(C4-Pad1)"))
+      (net 6 "Net-(C4-Pad1)"))
     (pad 2 thru_hole oval (at 2.54 0) (size 1.905 2) (drill 1.1) (layers *.Cu *.Mask)
       (net 1 GND))
@@
       (net 1 GND))
     (pad 2 thru_hole circle (at 3.81 0 270) (size 1.99898 1.99898) (drill 0.8001) (layers *.Cu *.Mask)
-      (net 5 "Net-(D1-Pad1)"))
+      (net 5 AC))
   )
   (module Capacitor_SMD:C_0805_2012Metric_Pad1.15x1.40mm_HandSolder (layer F.Cu)
@@
     )
     (pad 1 smd roundrect (at -1.025 0 90) (size 1.15 1.4) (layers F.Cu F.Paste F.Mask) (roundrect_rratio 0.217391)
-      (net 7 "Net-(C4-Pad1)"))
+      (net 6 "Net-(C4-Pad1)"))
     (pad 2 smd roundrect (at 1.025 0 90) (size 1.15 1.4) (layers F.Cu F.Paste F.Mask) (roundrect_rratio 0.217391)
       (net 1 GND))
@@
     )
     (pad 1 thru_hole rect (at 0 0 90) (size 2.2 2.2) (drill 1.1) (layers *.Cu *.Mask)
-      (net 5 "Net-(D1-Pad1)"))
+      (net 5 AC))
     (pad 2 thru_hole oval (at 7.62 0 90) (size 2.2 2.2) (drill 1.1) (layers *.Cu *.Mask)
-      (net 6 AC))
+      (net 7 "Net-(D1-Pad2)"))
     (model ${KISYS3DMOD}/Diode_THT.3dshapes/D_DO-41_SOD81_P7.62mm_Horizontal.wrl
       (at (xyz 0 0 0))
@@
     )
     (pad 1 thru_hole rect (at 0 0 180) (size 2.2 2.2) (drill 1.1) (layers *.Cu *.Mask)
-      (net 7 "Net-(C4-Pad1)"))
+      (net 6 "Net-(C4-Pad1)"))
     (pad 2 thru_hole oval (at 7.62 0 180) (size 2.2 2.2) (drill 1.1) (layers *.Cu *.Mask)
-      (net 6 AC))
+      (net 7 "Net-(D1-Pad2)"))
     (model ${KISYS3DMOD}/Diode_THT.3dshapes/D_DO-41_SOD81_P7.62mm_Horizontal.wrl
       (at (xyz 0 0 0))
@@
       (net 1 GND))
     (pad 1 thru_hole rect (at 0 0 270) (size 2.2 2.2) (drill 1.1) (layers *.Cu *.Mask)
-      (net 7 "Net-(C4-Pad1)"))
+      (net 6 "Net-(C4-Pad1)"))
     (model ${KISYS3DMOD}/Diode_THT.3dshapes/D_DO-41_SOD81_P7.62mm_Horizontal.wrl
       (at (xyz 0 0 0))
@@
     )
     (pad 1 thru_hole rect (at 0 0) (size 2.2 2.2) (drill 1.1) (layers *.Cu *.Mask)
-      (net 5 "Net-(D1-Pad1)"))
+      (net 5 AC))
     (pad 2 thru_hole oval (at 7.62 0) (size 2.2 2.2) (drill 1.1) (layers *.Cu *.Mask)
       (net 1 GND))
@@
   (segment (start 161.036 87.85949) (end 162.485491 89.308981) (width 0.5) (layer F.Cu) (net 1))
   (segment (start 161.036 86.36) (end 161.036 87.85949) (width 0.5) (layer F.Cu) (net 1) (status 10))
-  (segment (start 127 101.092) (end 127 96.012) (width 0.5) (layer F.Cu) (net 1))
-  (segment (start 127.032 101.124) (end 127 101.092) (width 0.5) (layer F.Cu) (net 1))
-  (segment (start 134.963856 101.124) (end 127.032 101.124) (width 0.5) (layer F.Cu) (net 1))
+  (segment (start 127 101.092) (end 127 96.012) (width 0.5) (layer F.Cu) (net 1) (status 30))
+  (segment (start 127.032 101.124) (end 127 101.092) (width 0.5) (layer F.Cu) (net 1) (status 30))
+  (segment (start 134.963856 101.124) (end 127.032 101.124) (width 0.5) (layer F.Cu) (net 1) (status 30))
   (segment (start 122.894 77.706) (end 117.54 77.706) (width 0.5) (layer F.Cu) (net 1))
   (segment (start 123.444 78.256) (end 122.894 77.706) (width 0.5) (layer F.Cu) (net 1))
-  (segment (start 117.54 77.706) (end 116.84 77.706) (width 0.5) (layer F.Cu) (net 1))
-  (segment (start 123.444 79.756) (end 123.444 78.256) (width 0.5) (layer F.Cu) (net 1))
-  (segment (start 116.14 77.706) (end 116.84 77.706) (width 0.5) (layer F.Cu) (net 1))
+  (segment (start 117.54 77.706) (end 116.84 77.706) (width 0.5) (layer F.Cu) (net 1) (status 20))
+  (segment (start 123.444 79.756) (end 123.444 78.256) (width 0.5) (layer F.Cu) (net 1) (status 10))
+  (segment (start 116.14 77.706) (end 116.84 77.706) (width 0.5) (layer F.Cu) (net 1) (status 30))
   (segment (start 130.505999 82.269999) (end 134.112 85.876) (width 0.5) (layer F.Cu) (net 1))
   (segment (start 125.910499 82.269999) (end 130.505999 82.269999) (width 0.5) (layer F.Cu) (net 1))
-  (segment (start 134.112 85.876) (end 134.112 87.376) (width 0.5) (layer F.Cu) (net 1))
-  (segment (start 123.444 79.8035) (end 125.910499 82.269999) (width 0.5) (layer F.Cu) (net 1))
-  (segment (start 123.444 79.756) (end 123.444 79.8035) (width 0.5) (layer F.Cu) (net 1))
+  (segment (start 134.112 85.876) (end 134.112 87.376) (width 0.5) (layer F.Cu) (net 1) (status 20))
+  (segment (start 123.444 79.8035) (end 125.910499 82.269999) (width 0.5) (layer F.Cu) (net 1) (status 10))
+  (segment (start 123.444 79.756) (end 123.444 79.8035) (width 0.5) (layer F.Cu) (net 1) (status 30))
   (segment (start 119.117998 89.916) (end 113.76749 89.916) (width 0.5) (layer B.Cu) (net 1))
-  (segment (start 113.76749 89.916) (end 112.268 89.916) (width 0.5) (layer B.Cu) (net 1))
+  (segment (start 113.76749 89.916) (end 112.268 89.916) (width 0.5) (layer B.Cu) (net 1) (status 20))
   (segment (start 125.213998 96.012) (end 119.117998 89.916) (width 0.5) (layer B.Cu) (net 1))
-  (segment (start 127 96.012) (end 125.213998 96.012) (width 0.5) (layer B.Cu) (net 1))
+  (segment (start 127 96.012) (end 125.213998 96.012) (width 0.5) (layer B.Cu) (net 1) (status 10))
   (segment (start 127.4365 79.756) (end 135.128 79.756) (width 0.5) (layer F.Cu) (net 2) (status 20))
   (segment (start 125.984 79.756) (end 127.4365 79.756) (width 0.5) (layer F.Cu) (net 2) (status 10))
@@
   (segment (start 143.002 99.314) (end 161.036 99.314) (width 0.5) (layer F.Cu) (net 4) (status 20))
   (segment (start 142.748 99.06) (end 143.002 99.314) (width 0.5) (layer F.Cu) (net 4))
-  (segment (start 119.38 97.104) (end 119.38 101.092) (width 0.5) (layer F.Cu) (net 5))
-  (segment (start 119.38 95.504) (end 119.38 97.104) (width 0.5) (layer F.Cu) (net 5))
+  (segment (start 119.38 97.104) (end 119.38 101.092) (width 0.5) (layer F.Cu) (net 5) (status 20))
+  (segment (start 119.38 95.504) (end 119.38 97.104) (width 0.5) (layer F.Cu) (net 5) (status 10))
   (segment (start 119.202 93.726) (end 119.38 93.904) (width 0.5) (layer F.Cu) (net 5))
-  (segment (start 119.38 93.904) (end 119.38 95.504) (width 0.5) (layer F.Cu) (net 5))
-  (segment (start 112.268 93.726) (end 119.202 93.726) (width 0.5) (layer F.Cu) (net 5))
-  (segment (start 119.38 87.884) (end 119.38 83.82) (width 0.5) (layer F.Cu) (net 6))
-  (segment (start 127 88.392) (end 127 83.82) (width 0.5) (layer F.Cu) (net 7))
-  (segment (start 120.904 79.756) (end 116.84 79.756) (width 0.5) (layer F.Cu) (net 7))
-  (segment (start 120.904 81.256) (end 120.904 79.756) (width 0.5) (layer F.Cu) (net 7))
-  (segment (start 123.468 83.82) (end 120.904 81.256) (width 0.5) (layer F.Cu) (net 7))
-  (segment (start 127 83.82) (end 123.468 83.82) (width 0.5) (layer F.Cu) (net 7))
+  (segment (start 119.38 93.904) (end 119.38 95.504) (width 0.5) (layer F.Cu) (net 5) (status 20))
+  (segment (start 112.268 93.726) (end 119.202 93.726) (width 0.5) (layer F.Cu) (net 5) (status 10))
+  (segment (start 119.38 87.884) (end 119.38 83.82) (width 0.5) (layer F.Cu) (net 7) (status 30))
+  (segment (start 127 88.392) (end 127 83.82) (width 0.5) (layer F.Cu) (net 6) (status 30))
+  (segment (start 120.904 79.756) (end 116.84 79.756) (width 0.5) (layer F.Cu) (net 6) (status 30))
+  (segment (start 120.904 81.256) (end 120.904 79.756) (width 0.5) (layer F.Cu) (net 6) (status 20))
+  (segment (start 123.468 83.82) (end 120.904 81.256) (width 0.5) (layer F.Cu) (net 6))
+  (segment (start 127 83.82) (end 123.468 83.82) (width 0.5) (layer F.Cu) (net 6) (status 10))
 )

Commit message: Better footprints and fixed pcb
Parts:
- removed the C4 at (116.8, 78.7)
- added C1: 100n, Capacitor_THT:C_Rect_L4.0mm_W2.5mm_P2.50mm, F.Cu at (113.3, 81.8)
- added C2: 100n, Capacitor_THT:C_Rect_L4.0mm_W2.5mm_P2.50mm, F.Cu at (131.6, 84.3)
- renumbered C1 to C3, C2 to C4, C3 to C5, J3 to J1, J1 to J2, J2 to J3
Connections:
- C3 pad 1: GND -> Net-(C1-Pad2)
- C4 pad 1: GND -> Net-(C1-Pad2)
- C5 pad 1: GND -> Net-(C1-Pad2)
- D1 pad 1: AC -> Net-(C1-Pad1)
- D1 pad 2: Net-(D1-Pad2) -> AC
- D2 pad 1: AC -> Net-(C1-Pad1)
- D3 pad 1: Net-(C4-Pad1) -> Net-(C1-Pad2)
- D3 pad 2: Net-(D1-Pad2) -> AC
- D4 pad 1: Net-(C4-Pad1) -> Net-(C1-Pad2)
- J2 pad 1: GND -> Net-(C1-Pad2)
- J3 pad 1: GND -> Net-(C1-Pad2)
- U1 pad 1: Net-(C4-Pad1) -> Net-(C1-Pad1)
- U1 pad 2: GND -> Net-(C1-Pad2)
Routing:
- net GND: track 115.2 -> 22.4 mm
- net Net-(C1-Pad2): track 0.00 -> 92.7 mm
- net Net-(C1-Pad1): track 0.00 -> 44.6 mm
- net Net-(C4-Pad1): track 17.3 -> 0.00 mm
- net Net-(C2-Pad2): track 29.8 -> 34.2 mm
- net Net-(D1-Pad2): track 4.06 -> 0.00 mm
- net AC: track 14.4 -> 13.6 mm

Commit message: Rev 2. Sigh.
Parts:
- R1, R2: footprint Resistor_THT:R_Axial_DIN0414_L11.9mm_D4.5mm_P7.62mm_Vertical -> Resistor_THT:R_Axial_DIN0414_L11.9mm_D4.5mm_P15.24mm_Horizontal
- moved J3 9.65 mm to (161.0, 96.0)
- moved J2 9.14 mm to (161.0, 86.4)
- moved R2 6.91 mm to (149.4, 77.7)
- moved R1 2.74 mm to (156.0, 96.0)
Routing:
- net Net-(C2-Pad2): track 34.2 -> 30.0 mm
- net Net-(C5-Pad2): track 44.9 -> 49.0 mm
- net Net-(C1-Pad2): track 92.7 -> 94.7 mm

Commit message: Add P4
Parts:
- moved D3 7.64 mm to (119.4, 84.3), turned to 0 degrees
- moved D4 7.11 mm to (127.0, 95.5), turned to 90 degrees
Connections:
- D3 pad 1: Net-(C1-Pad2) -> AC
- D3 pad 2: AC -> Net-(C1-Pad2)
- D4 pad 1: Net-(C1-Pad2) -> GND
- D4 pad 2: GND -> Net-(C1-Pad2)
Routing:
- net Net-(C1-Pad2): track 94.7 -> 92.4 mm
- net GND: track 22.4 -> 23.3 mm
- net AC: track 13.6 -> 13.1 mm
