File: P4/P4.sch (KiCad schematic (older format))
At the start: 12 parts, among them J1 RPi_GPIO, U1 PGA2310

Commit message: Add connections for rotary encoder, display and power relay
Parts:
- added J2: Conn_02x10_Odd_Even, Connector_PinHeader_2.54mm:PinHeader_2x10_P2.54mm_Vertical, symbol Connector_Generic:Conn_02x10_Odd_Even
- added J3: Conn_01x05_Male, Connector_PinSocket_2.54mm:PinSocket_1x05_P2.54mm_Vertical, symbol Connector:Conn_01x05_Male
- added J4: Conn_01x02_Male, Connector_PinSocket_2.54mm:PinSocket_1x02_P2.54mm_Vertical, symbol Connector:Conn_01x02_Male
Connections:
- net labels added: #EPD_CS, +3.3V
- wire segments 90 -> 100
Changed lines of the file:
@@
 Wire Wire Line
 	1700 1100 1500 1100
+$Comp
+L Connector:Conn_01x05_Male J3
+U 1 1 64B816F1
+P 9800 1400
+F 0 "J3" H 9908 1781 50  0000 C CNN
+F 1 "Conn_01x05_Male" H 9908 1690 50  0000 C CNN
+F 2 "Connector_PinSocket_2.54mm:PinSocket_1x05_P2.54mm_Vertical" H 9800 1400 50  0001 C CNN
+F 3 "~" H 9800 1400 50  0001 C CNN
+	1    9800 1400
+	1    0    0    -1
+$EndComp
+$Comp
+L power:GND #PWR0108
+U 1 1 64B902F0
+P 8100 900
+F 0 "#PWR0108" H 8100 650 50  0001 C CNN
+F 1 "GND" H 8105 727 50  0000 C CNN
+F 2 "" H 8100 900 50  0001 C CNN
+F 3 "" H 8100 900 50  0001 C CNN
+	1    8100 900
+	-1   0    0    1
+$EndComp
+$Comp
+L power:+3.3V #PWR0109
+U 1 1 64B85CA6
+P 7400 2350
+F 0 "#PWR0109" H 7400 2200 50  0001 C CNN
+F 1 "+3.3V" H 7415 2523 50  0000 C CNN
+F 2 "" H 7400 2350 50  0001 C CNN
+F 3 "" H 7400 2350 50  0001 C CNN
+	1    7400 2350
+	1    0    0    -1
+$EndComp
+$Comp
+L power:+3.3V #PWR0110
+U 1 1 64B86109
+P 10000 1200
+F 0 "#PWR0110" H 10000 1050 50  0001 C CNN
+F 1 "+3.3V" V 10015 1328 50  0000 L CNN
+F 2 "" H 10000 1200 50  0001 C CNN
+F 3 "" H 10000 1200 50  0001 C CNN
+	1    10000 1200
+	0    1    1    0
+$EndComp
+$Comp
+L power:GND #PWR0111
+U 1 1 64B86733
+P 10000 1300
+F 0 "#PWR0111" H 10000 1050 50  0001 C CNN
+F 1 "GND" H 10005 1127 50  0000 C CNN
+F 2 "" H 10000 1300 50  0001 C CNN
+F 3 "" H 10000 1300 50  0001 C CNN
+	1    10000 1300
+	0    -1   -1   0
+$EndComp
+Wire Wire Line
+	9300 3050 10000 3050
+Wire Wire Line
+	10000 3050 10000 1600
+Wire Wire Line
+	10000 1500 10100 1500
+Wire Wire Line
+	10100 1500 10100 3150
+Wire Wire Line
+	10100 3150 9300 3150
+Wire Wire Line
+	10000 1400 10200 1400
+Wire Wire Line
+	10200 1400 10200 3250
+Wire Wire Line
+	10200 3250 9300 3250
+$Comp
+L Connector:Conn_01x02_Male J4
+U 1 1 64B917D8
+P 9950 3700
+F 0 "J4" H 10058 3881 50  0000 C CNN
+F 1 "Conn_01x02_Male" H 10058 3790 50  0000 C CNN
+F 2 "Connector_PinSocket_2.54mm:PinSocket_1x02_P2.54mm_Vertical" H 9950 3700 50  0001 C CNN
+F 3 "~" H 9950 3700 50  0001 C CNN
+	1    9950 3700
+	1    0    0    -1
+$EndComp
+$Comp
+L power:+5V #PWR0112
+U 1 1 64B9214C
+P 10150 3700
+F 0 "#PWR0112" H 10150 3550 50  0001 C CNN
+F 1 "+5V" H 10165 3873 50  0000 C CNN
+F 2 "" H 10150 3700 50  0001 C CNN
+F 3 "" H 10150 3700 50  0001 C CNN
+	1    10150 3700
+	1    0    0    -1
+$EndComp
+Wire Wire Line
+	9300 4050 10150 4050
+Wire Wire Line
+	10150 4050 10150 3800
+$Comp
+L Connector_Generic:Conn_02x10_Odd_Even J2
+U 1 1 64B9CA24
+P 7600 1200
+F 0 "J2" V 7696 612 50  0000 R CNN
+F 1 "Conn_02x10_Odd_Even" V 7605 612 50  0000 R CNN
+F 2 "Connector_PinHeader_2.54mm:PinHeader_2x10_P2.54mm_Vertical" H 7600 1200 50  0001 C CNN
+F 3 "~" H 7600 1200 50  0001 C CNN
+	1    7600 1200
+	0    -1   -1   0
+$EndComp
+$Comp
+L power:+3.3V #PWR0113
+U 1 1 64BA6ECD
+P 7200 1400
+F 0 "#PWR0113" H 7200 1250 50  0001 C CNN
+F 1 "+3.3V" H 7215 1573 50  0000 C CNN
+F 2 "" H 7200 1400 50  0001 C CNN
+F 3 "" H 7200 1400 50  0001 C CNN
+	1    7200 1400
+	-1   0    0    1
+$EndComp
+Text GLabel 7900 1400 3    50   Input ~ 0
+MOSI
+Text GLabel 7800 900  1    50   Input ~ 0
+MISO
+Text GLabel 7400 3950 0    50   Input ~ 0
+#EPD_CS
+Text GLabel 8100 1400 3    50   Input ~ 0
+#EPD_CS
+$Comp
+L power:GND #PWR0115
+U 1 1 64BD06D8
+P 7400 4250
+F 0 "#PWR0115" H 7400 4000 50  0001 C CNN
+F 1 "GND" H 7405 4077 50  0000 C CNN
+F 2 "" H 7400 4250 50  0001 C CNN
+F 3 "" H 7400 4250 50  0001 C CNN
+	1    7400 4250
+	1    0    0    -1
+$EndComp
 $EndSCHEMATC

Commit message: Add transistors for relays
Parts:
- added Q1, Q2, Q3, Q4: Q_NPN_BEC, Package_TO_SOT_SMD:SOT-23W_Handsoldering, symbol Device:Q_NPN_BEC
- added R1, R2, R3, R4: 1k, Resistor_SMD:R_0603_1608Metric_Pad0.98x0.95mm_HandSolder, symbol Device:R
Connections:
- net labels added: RL1, RL2, RL3, RL4
- wire segments 100 -> 94

Commit message: Guarduino switched to MCP3008, PCB not done
Parts:
- U1: footprint Package_SO:SOIC-16_3.9x9.9mm_P1.27mm -> Package_SO:SOIC-16W_7.5x10.3mm_P1.27mm
Connections:
- net labels added: CD|Aux_L, CD|Aux_R, OutL, OutR, VCL, VCR
- wire segments 94 -> 69
Changed lines of the file:
@@
 F 0 "U1" H 2325 2881 50  0000 C CNN
 F 1 "PGA2310" H 2325 2790 50  0000 C CNN
-F 2 "Package_SO:SOIC-16_3.9x9.9mm_P1.27mm" H 2350 1900 50  0001 C CNN
+F 2 "Package_SO:SOIC-16W_7.5x10.3mm_P1.27mm" H 2350 1900 50  0001 C CNN
 F 3 "http://www.ti.com/lit/ds/symlink/pga2310.pdf" H 2350 1900 50  0001 C CNN
 	1    2350 1900
@@
 	3350 4850 1450 4850
 Wire Wire Line
-	4900 4250 4600 4250
-Wire Wire Line
-	4600 4250 4600 5800
-Wire Wire Line
-	4900 4650 4900 5700
-Wire Wire Line
-	5700 7150 5550 7150
-Wire Wire Line
 	1450 6000 5600 6000
 Wire Wire Line
@@
 Wire Wire Line
 	5600 6750 5550 6750
-Wire Wire Line
-	1450 6200 5700 6200
-Wire Wire Line
-	5700 6200 5700 7150
-Wire Wire Line
-	5550 6950 5850 6950
-Wire Wire Line
-	5850 6950 5850 5800
-Wire Wire Line
-	4600 5800 5850 5800
-Wire Wire Line
-	6000 5700 6000 7350
-Wire Wire Line
-	5550 7350 6000 7350
-Wire Wire Line
-	4900 5700 6000 5700
 $Comp
 L Connector:Conn_01x03_Male +-12V1
@@
 	1500 900  2250 900
 Wire Wire Line
-	1500 1000 1600 1000
-Wire Wire Line
-	1600 1000 1600 1600
-Wire Wire Line
-	1600 1600 1750 1600
-Wire Wire Line
-	1750 2200 1600 2200
-Wire Wire Line
-	1600 2200 1600 1600
-Connection ~ 1600 1600
+	1500 1000 1550 1000
 $Comp
 L power:GND #PWR?
@@
 	1    0    0    -1
 $EndComp
-Wire Wire Line
-	1500 7300 2100 7300
-Wire Wire Line
-	2100 7300 2100 3100
-Wire Wire Line
-	2100 3100 1200 3100
-Wire Wire Line
-	1200 3100 1200 1800
-Wire Wire Line
-	1200 1800 1750 1800
 $Comp
 L lci-kicad:Omron_G6K RL?
@@
 $EndComp
 Wire Wire Line
-	1450 6850 4150 6850
-Wire Wire Line
-	4000 6650 1450 6650
-Wire Wire Line
 	1450 4150 3900 4150
 Wire Wire Line
 	1450 3950 3750 3950
 Wire Wire Line
-	3900 4150 3900 2250
-Wire Wire Line
-	3750 3950 3750 1850
-Wire Wire Line
-	3900 2250 4850 2250
-Wire Wire Line
-	3750 1850 4850 1850
-Wire Wire Line
-	4150 2800 5800 2800
-Wire Wire Line
-	5650 2650 4000 2650
-Wire Wire Line
-	4000 2650 4000 6650
-Wire Wire Line
 	5450 1750 5650 1750
 Wire Wire Line
-	5650 1750 5650 2650
-Wire Wire Line
 	5450 2150 5800 2150
-Wire Wire Line
-	5800 2150 5800 2800
-Wire Wire Line
-	1700 2000 1400 2000
-Wire Wire Line
-	1400 2000 1400 2950
-Wire Wire Line
-	1400 2950 2200 2950
-Wire Wire Line
-	2200 2950 2200 7500
-Wire Wire Line
-	2200 7500 1500 7500
 Text Label 2700 3950 0    50   ~ 0
 Phono_in_L
@@
 Text Label 2800 6200 0    50   ~ 0
 RPI_out_R
-Text Label 2800 6650 0    50   ~ 0
+Text Label 1450 6650 0    50   ~ 0
 RPi_in_L
-Text Label 2800 6850 0    50   ~ 0
+Text Label 1450 6850 0    50   ~ 0
 RPi_in_R
-Text Label 4950 6850 2    50   ~ 0
-INL
-Text Label 4950 7250 2    50   ~ 0
-INR
-Text GLabel 5450 1950 2    50   Input ~ 0
-INL
-Text GLabel 1750 1400 0    50   Input ~ 0
-INL
-Text GLabel 5450 2350 2    50   Input ~ 0
-INR
-Text GLabel 1750 2400 0    50   Input ~ 0
-INR
 Text GLabel 2900 1400 2    50   Input ~ 0
 #MUTE
@@
 $EndComp
 Wire Wire Line
-	4150 2800 4150 6850
-Wire Wire Line
 	4900 3850 4500 3850
 Text GLabel 7400 3050 0    50   Input ~ 0
@@
 Wire Wire Line
 	6900 2750 7400 2750
+Wire Wire Line
+	3900 4150 3900 3200
+Wire Wire Line
+	3900 3200 5800 3200
+Wire Wire Line
+	5800 3200 5800 2150
+Wire Wire Line
+	3750 3950 3750 3000
+Wire Wire Line
+	3750 3000 5650 3000
+Wire Wire Line
+	5650 3000 5650 1750
+Wire Wire Line
+	6000 6200 6000 7150
+Wire Wire Line
+	6000 7150 5550 7150
+Wire Wire Line
+	1450 6200 6000 6200
+Text Label 4900 4250 2    50   ~ 0
+CD|Aux_L
+Text Label 4900 4650 2    50   ~ 0
+CD|Aux_R
+Text Label 5450 1950 0    50   ~ 0
+CD|Aux_L
+Text Label 5450 2350 0    50   ~ 0
+CD|Aux_R
+Text Label 4850 1850 2    50   ~ 0
+INL
+Text Label 4850 2250 2    50   ~ 0
+INR
+Text Label 1500 7300 0    50   ~ 0
+OutL
+Text Label 1500 7500 0    50   ~ 0
+OutR
+Text Label 1750 2000 2    50   ~ 0
+OutR
+Text Label 1750 1800 2    50   ~ 0
+OutL
+Wire Wire Line
+	1550 1000 1550 1600
+Wire Wire Line
+	1550 2200 1750 2200
+Wire Wire Line
+	1550 1600 1750 1600
+Connection ~ 1550 1600
+Wire Wire Line
+	1550 1600 1550 2200
+Text Label 5550 7350 0    50   ~ 0
+INR
+Text Label 5550 6950 0    50   ~ 0
+INL
+Text Label 1750 1400 2    50   ~ 0
+VCL
+Text Label 1750 2400 2    50   ~ 0
+VCR
+Text Label 4950 6850 2    50   ~ 0
+VCL
+Text Label 4950 7250 2    50   ~ 0
+VCR
 $EndSCHEMATC
