File: garduino/garduino.kicad_sch (KiCad schematic)
At the start: 38 parts, among them J1 ADC0, J10 OUT6, J11 ADC6, J12 OUT5, J13 OUT4, J14 DIN, J15 OUT3, J16 12v, J17 OUT2, J18 OUT1, J19 RPi, J2 ADC1, J20 ADC7, J21 OUT1, J22 ADC8, J23 ADC9, J3 ADC2, J4 OUT1, J5 ADC3, J6 ADC4, J7 OUT8, J8 OUT7, J9 ADC5, Q1 NCV8403, Q12 NCV8403, Q2 NCV8403, Q3 NCV8403, Q4 NCV8403, Q5 NCV8403, Q6 NCV8403, Q7 NCV8403, Q8 NCV8403, Q9 NCV8403, U1 MCP3008

Commit message: Cleanups, placement might work
Parts:
- removed J14: DIN, Connector_PinSocket_2.54mm:PinSocket_1x02_P2.54mm_Vertical, symbol Connector_Generic:Conn_01x02
- J10: renamed from J8; value OUT7 -> OUT6
- J11: renamed from J7; value OUT8 -> OUT7
- J12: renamed from J21; value OUT1 -> OUT8
- J13: renamed from J4; value OUT1 -> OUT9
- J4: renamed from J18; value OUT1 -> OUT0
- J5: renamed from J17; value OUT2 -> OUT1
- J6: renamed from J15; value OUT3 -> OUT2
- J7: renamed from J13; value OUT4 -> OUT3
- J8: renamed from J12; value OUT5 -> OUT4
- J9: renamed from J10; value OUT6 -> OUT5
- renumbered C4 to C1, C5 to C2, D9 to D1, J19 to J1, J1 to J14, J2 to J15, J3 to J16, J5 to J17, J6 to J18, J9 to J19, J11 to J20, J20 to J21, J16 to J3, Q9 to Q10, Q6 to Q2, Q2 to Q3, Q7 to Q4, Q12 to Q5, Q3 to Q6, Q4 to Q7, Q5 to Q9, R14 to R1
Other:
- moved on the sheet: J13

Commit message: Routing done (not pretty)
Parts:
- removed J12: OUT8, Connector_PinSocket_2.54mm:PinSocket_1x02_P2.54mm_Vertical, symbol Connector_Generic:Conn_01x02
- removed J13: OUT9, Connector_PinSocket_2.54mm:PinSocket_1x02_P2.54mm_Vertical, symbol Connector_Generic:Conn_01x02
- removed J22: ADC8, Connector_PinHeader_2.54mm:PinHeader_1x03_P2.54mm_Vertical, symbol Connector_Generic:Conn_01x03
- removed J23: ADC9, Connector_PinHeader_2.54mm:PinHeader_1x03_P2.54mm_Vertical, symbol Connector_Generic:Conn_01x03
- removed Q10, Q8: NCV8403, Package_TO_SOT_SMD:TO-252-2, symbol Transistor_FET:IPD50R3K0CE
Connections:
- net GPIO26: now also Q2.1 (G)
- net GPIO6: no longer Q2.1 (G)

Commit message: Add capacitors for 3.3v
Parts:
- added C3: 1mF, Capacitor_THT:C_Rect_L4.0mm_W2.5mm_P2.50mm, symbol Device:C_Small
- added C4: 100nF, Capacitor_SMD:C_0603_1608Metric_Pad1.08x0.95mm_HandSolder, symbol Device:C_Small
Connections:
- net +3.3V: now also C3.2, C4.2
- net GND: now also C3.1, C4.1
