File: garduino/garduino.kicad_pcb (KiCad board)
At the start: 2 copper layers, 65 x 56 mm, 41 parts, among them J1 RPi, J10 OUT6, J11 OUT7, J12 OUT8, J13 OUT9, J14 ADC0, J15 ADC1, J16 ADC2, J17 ADC3, J18 ADC4, J19 ADC5, J20 ADC6, J21 ADC7, J22 ADC8, J23 ADC9, J3 12v, J4 OUT0, J5 OUT1, J6 OUT2, J7 OUT3, J8 OUT4, J9 OUT5, Q1 NCV8403, Q10 NCV8403, Q2 NCV8403, Q3 NCV8403, Q4 NCV8403, Q5 NCV8403, Q6 NCV8403, Q7 NCV8403, Q8 NCV8403, Q9 NCV8403, U1 MCP3008

Commit message: Routing done (not pretty)
Parts:
- removed J12: OUT8, Connector_PinSocket_2.54mm:PinSocket_1x02_P2.54mm_Vertical
- removed J13: OUT9, Connector_PinSocket_2.54mm:PinSocket_1x02_P2.54mm_Vertical
- removed J22: ADC8, Connector_PinHeader_2.54mm:PinHeader_1x03_P2.54mm_Vertical
- removed J23: ADC9, Connector_PinHeader_2.54mm:PinHeader_1x03_P2.54mm_Vertical
- removed Q10, Q8: NCV8403, Package_TO_SOT_SMD:TO-252-2
Connections:
- Q2 pad 1: /GPIO6 -> /GPIO26
Routing:
- net +5V: track 24.1 -> 141.2 mm, vias 0 -> 3
- net /GPIO26: track 0.00 -> 70.8 mm
- net GND: track 179.0 -> 248.3 mm, vias 6 -> 10
- net /GPIO5: track 0.00 -> 63.6 mm
- net /GPIO0: track 0.00 -> 63.1 mm
- net /GPIO27: track 0.00 -> 50.4 mm
- net /GPIO22: track 0.00 -> 49.1 mm
- net +3.3V: track 0.00 -> 40.4 mm, vias 0 -> 2
- net /GPIO23: track 0.00 -> 33.1 mm
- net /SPI0_MOSI: track 0.00 -> 32.8 mm, vias 0 -> 1
- net /OUT6: track 0.00 -> 32.6 mm, vias 0 -> 2
- net /OUT7: track 0.00 -> 31.5 mm, vias 0 -> 2
- net /GPIO24: track 0.00 -> 31.0 mm
- net /CH7: track 0.00 -> 29.1 mm
- net /CH6: track 0.00 -> 26.0 mm
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Other:
- outline, holes or cut-outs redrawn

Commit message: Add capacitors for 3.3v
Parts:
- added C3: 1mF, Capacitor_THT:C_Rect_L4.0mm_W2.5mm_P2.50mm, F.Cu at (112.5, 101.2)
- added C4: 100nF, Capacitor_SMD:C_0603_1608Metric_Pad1.08x0.95mm_HandSolder, F.Cu at (113.1, 104.5)
Routing:
- net +3.3V: track 40.4 -> 81.1 mm
- net GND: track 248.3 -> 259.1 mm

Commit message: Add label
Parts:
- J3: value 12v -> 12v+
Other:
- board text added: "waterpi 1.0"
- board text removed: "+"
Changed lines of the file:
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@@
 			)
 		)
-		(property "Value" "12v"
-			(at 0 5.31 0)
+		(property "Value" "12v+"
+			(at 0.048 5.174 0)
 			(layer "F.SilkS")
 			(effects
@@
 			(at 0 -4.5 90)
 			(layer "F.SilkS")
+			(hide yes)
 			(effects
 				(font
@@
 			(at 0 -4.5 90)
 			(layer "F.SilkS")
+			(hide yes)
 			(effects
 				(font
@@
 			(at 0 -4.5 90)
 			(layer "F.SilkS")
+			(hide yes)
 			(effects
 				(font
@@
 			(at 0 -4.5 90)
 			(layer "F.SilkS")
+			(hide yes)
 			(effects
 				(font
@@
 			(at 0 -4.5 90)
 			(layer "F.SilkS")
+			(hide yes)
 			(effects
 				(font
@@
 			(at 0 -4.5 90)
 			(layer "F.SilkS")
+			(hide yes)
 			(effects
 				(font
@@
 			(at 0 -4.5 90)
 			(layer "F.SilkS")
+			(hide yes)
 			(effects
 				(font
@@
 			(at 0 -4.5 90)
 			(layer "F.SilkS")
+			(hide yes)
 			(effects
 				(font
@@
 		(layer "Edge.Cuts")
 	)
-	(gr_text "+"
-		(at 92.202 128.778 0)
+	(gr_text "waterpi 1.0"
+		(at 96 97.75 270)
 		(layer "F.SilkS")
 		(effects
@@
 				(size 1.5 1.5)
 				(thickness 0.3)
+				(bold yes)
 			)
+			(justify left bottom)
 		)
 	)
