File: waterpi/waterpi.kicad_pcb (KiCad board)
At the start: 2 copper layers, 65 x 56 mm, 37 parts, among them J1 RPi, J10 OUT6, J11 OUT7, J14 ADC0, J15 ADC1, J16 ADC2, J17 ADC3, J18 ADC4, J19 ADC5, J20 ADC6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

Commit message: Add connector for display
Parts:
- added J2: Conn_01x10, Connector_PinSocket_2.54mm:PinSocket_1x10_P2.54mm_Vertical, F.Cu at (100.2, 101.3)
- J3: value 12v+ -> 12v
Routing:
- net /SPI1_MOSI: track 0.00 -> 73.2 mm
- net /SPI1_MISO: track 0.00 -> 69.5 mm, vias 0 -> 1
- net /PWM0: track 0.00 -> 55.6 mm
- net /GPIO25: track 0.00 -> 33.3 mm, vias 0 -> 1
- net /SPI1_CE0: track 0.00 -> 28.6 mm
- net /GPIO27: track 50.4 -> 59.5 mm
- net GND: track 259.1 -> 267.6 mm
- net +3.3V: track 81.1 -> 85.5 mm
- net /SPI0_MOSI: track 32.8 -> 29.9 mm

Commit message: GND connections/warnings
Routing:
- net GND: track 267.6 -> 305.8 mm, vias 10 -> 13
- net +12V: track 11.7 -> 46.7 mm
- net /GPIO5: track 63.6 -> 64.4 mm
- net +5V: track 141.2 -> 140.7 mm
